File: Syml-PCB.sch (KiCad schematic (older format))
At the start: 1 part

Commit message: Kira componenets added
Parts:
- removed U?: ATSAM4S8CA-CU, BGA100C80P10X10_900X900X110, symbol Kira:ATSAM4S8CA-CU
Connections:
- net labels removed: +5V
Changed lines of the file:
@@
 EESchema Schematic File Version 4
-EELAYER 26 0
+LIBS:Syml-PCB-cache
+EELAYER 29 0
 EELAYER END
 $Descr A4 11693 8268
@@
 Comment4 ""
 $EndDescr
-$Comp
-L Kira:ATSAM4S8CA-CU U?
-U 1 1 5CCCF66E
-P 2325 3575
-F 0 "U?" H 2325 6345 50  0000 C CNN
-F 1 "ATSAM4S8CA-CU" H 2325 6254 50  0000 C CNN
-F 2 "BGA100C80P10X10_900X900X110" H 2325 3575 50  0001 L BNN
-F 3 "Microchip" H 2325 3575 50  0001 L BNN
-	1    2325 3575
-	1    0    0    -1
-$EndComp
-$Comp
-L power:+5V #PWR?
-U 1 1 5CCCF83F
-P 3775 900
-F 0 "#PWR?" H 3775 750 50  0001 C CNN
-F 1 "+5V" H 3790 1073 50  0000 C CNN
-F 2 "" H 3775 900 50  0001 C CNN
-F 3 "" H 3775 900 50  0001 C CNN
-	1    3775 900
-	1    0    0    -1
-$EndComp
 $EndSCHEMATC
