File: Syml-PCB.sch (KiCad schematic (older format))
At the start: 13 parts

Commit message: Add submodules
Parts:
- added A1, Apostrophe1, B1, BSlash1, Back1, Back2, C1, Comma1, D1, DArrow1, Del1, E1, Enter1, Equal1, Esc1, F0, F1, F10, F11, F12, F2, F3, F4, F5, F6, F7, F8, F9, G1, H1, Home1, I1, J1, K1, L1, LArrow1, LBracket1, LShift2, M1, MX0, MX1, MX2, MX3, MX4, MX5, MX6, MX7, MX8, MX9, Minus1, N1, O1, P1, Period1, PgDn1, PgUp1, Q1, R1, RArrow1, RBracket1, S1, Semicolon1, T1, TArrow1, Tilda1, U1, V1, W1, X1, Y1, Z1: MX-1U, MX_Alps_Hybrid:MX-1U, symbol MX_Alps_Hybrids:MX-1U
- added CLF1: 1800mA, Fuse:Fuse_1206_3216Metric, symbol Device:Polyfuse_Small
- added CapsLock1, RShift1: MX-1U, MX_Alps_Hybrid:MX-1.75U, symbol MX_Alps_Hybrids:MX-1U
- added D10, D11, D12, D13, D14, D15, D16, D17, D18, D19, D2, D20, D21, D22, D23, D24, D25, D26, D27, D28, D29, D3, D30, D31, D32, D33, D34, D35, D36, D37, D38, D39, D4, D40, D41, D42, D43, D44, D45, D46, D47, D48, D49, D5, D50, D51, D52, D53, D54, D55, D56, D57, D58, D59, D6, D60, D61, D62, D63, D64, D65, D66, D67, D68, D69, D7, D70, D71, D72, D73, D74, D75, D76, D77, D78, D79, D8, D80, D81, D82, D83, D84, D9: SOD-123, random-keyboard-parts:D_SOD-123-Pretty, symbol Device:D_Small
- added Enter2: MX-1U, MX_Alps_Hybrid:MX-2.25U, symbol MX_Alps_Hybrids:MX-1U
- added FSlash1, RAlt1, RCtrl1, Tab1: MX-1U, MX_Alps_Hybrid:MX-1.5U, symbol MX_Alps_Hybrids:MX-1U
- added LAlt1, LCtrl1, LShift1, LWK1: MX-1U, MX_Alps_Hybrid:MX-1.25U, symbol MX_Alps_Hybrids:MX-1U
- added R3: 10k, Resistor_SMD:R_0805_2012Metric, symbol Device:R_Small
- added R4, R6: 5.1k, Resistor_SMD:R_0805_2012Metric, symbol Device:R_Small
- added Space1: MX-1U, MX_Alps_Hybrid:MX-6.25U-ReversedStabilizers, symbol MX_Alps_Hybrids:MX-1U
- added U3, U4: IS31FL3733, Package_QFP:TQFP-48-1EP_7x7mm_P0.5mm_EP5x5mm, symbol random-keyboard-parts:IS31FL3733
- added USB1: 12401598E4#2A, Type-C:12401598E4#2A, symbol Type-C:12401598E4#2A
- C2, C3, C4, C5, C6, C7, C8: renamed from C?; footprint (none) -> Capacitor_SMD:C_0805_2012Metric
- R2, R5, R7: renamed from R?; footprint (none) -> Resistor_SMD:R_0805_2012Metric
- SW1: renamed from SW?; footprint (none) -> random-keyboard-parts:SKQG-1155865
- Y2: renamed from Y?; footprint (none) -> Crystal:Crystal_SMD_3225-4Pin_3.2x2.5mm
- gave numbers to parts that had none: 1
Connections:
- net labels added: COL0, COL1, COL10, COL11, COL12, COL13, COL14, COL15, COL2, COL3, COL4, COL5, COL6, COL7, COL8, COL9, D+, D-, ROW0, ROW1, ROW2, ROW3, ROW4, ROW5, VCC
- wire segments 60 -> 454
Other:
- moved on the sheet: C2, C3, C4, C5, C6, C7, C8, R2, R5, R7, SW1, U2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

Commit message: LED Controllers built
Parts:
- removed CLF1: 1800mA, Fuse:Fuse_1206_3216Metric, symbol Device:Polyfuse_Small
- removed R4, R6: 5.1k, Resistor_SMD:R_0805_2012Metric, symbol Device:R_Small
- removed USB1: 12401598E4#2A, Type-C:12401598E4#2A, symbol Type-C:12401598E4#2A
- added C? (x8): 0.47uF, symbol Device:C_Small
- added C? (x6): 0.1uF, symbol Device:C_Small
- added J?: Connector_Generic_Conn_01x04, symbol Unified-Daughterboard-cache:Connector_Generic_Conn_01x04
- added J? (x4): Connector_Generic_Conn_01x01, symbol Unified-Daughterboard-cache:Connector_Generic_Conn_01x01
- added R? (x2): 5.1k, symbol Device:R_Small
- added R? (x2): 20k, symbol Device:R_Small
- added R? (x4): 100k, symbol Device:R_Small
- added R? (x4): 1k, symbol Device:R_Small
- added USB?: Type-C_HRO-TYPE-C-31-M-12, symbol Unified-Daughterboard-cache:Type-C_HRO-TYPE-C-31-M-12
Connections:
- net +5V: now also U3.20 (PVCC), U3.29 (PVCC), U3.37 (AVCC), U3.38 (DVCC), U4.20 (PVCC), U4.29 (PVCC), U4.37 (AVCC), U4.38 (DVCC), C?.1, C?.1, C?.1, C?.1, C?.1, C?.1, C?.1, C?.1, C?.1, C?.1, C?.1, C?.1, R?.1, R?.1, R?.1, R?.1
- net D+: now also J?.3 (Pin_3), USB?.6 (DP1), USB?.8 (DP2)
- net D-: now also J?.2 (Pin_2), USB?.5 (DN2), USB?.7 (DN1)
- net GND: now also U3.43 (ADDR1), U3.44 (ADDR2), U3.48 (GND), U4.43 (ADDR1), U4.44 (ADDR2), U4.48 (GND), C?.2, C?.2, C?.2, C?.2, C?.2, C?.2, C?.2, C?.2, C?.2, C?.2, C?.2, C?.2, C?.2, C?.2, J?.1 (Pin_1), J?.1 (Pin_1), J?.1 (Pin_1), J?.1 (Pin_1), J?.4 (Pin_4), R?.2, R?.2, R?.2, R?.2, R?.2, R?.2, R?.2, R?.2, USB?.1 (GND), USB?.12 (GND), USB?.13 (SHIELD)
- net VCC: now also J?.1 (Pin_1), USB?.11 (VBUS), USB?.2 (VBUS)
- net at U4.35 (RSET): now also R?.1
- net at U4.39 (VIO): now also C?.1
- net SYNC: now reaches U4.40 (SYNC)
- net SYNC: now also U3.40 (SYNC)
- net SDA1: now reaches U4.41 (SDA)
- net SDA1: now also R?.2
- net SCL1: now reaches U4.42 (SCL)
- net SCL1: now also R?.2
- net SDB1: now reaches U4.46 (SDB)
- net SDB1: now also R?.1
- net IICRST: now reaches U4.47 (IICRST)
- net IICRST: now also U3.47 (IICRST), R?.1, R?.1
- net at U3.35 (RSET): now also R?.1
- net at U3.39 (VIO): now also C?.1
- net SDA0: now reaches U3.41 (SDA)
- net SDA0: now also R?.2
- net SCL0: now reaches U3.42 (SCL)
- net SCL0: now also R?.2
- net SDB0: now reaches U3.46 (SDB)
- net SDB0: now also R?.1
- new net: R?.1, USB?.10 (CC2)
- new net: R?.1, USB?.4 (CC1)
Other:
- moved on the sheet: A1, Apostrophe1, B1, BSlash1, Back1, Back2, C1, C2, C3, C4, C5, C6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

Commit message: PCB Complete
Parts:
- removed C? (x8): 0.47uF, symbol Device:C_Small
- removed C? (x6): 0.1uF, symbol Device:C_Small
- removed D70: SOD-123, random-keyboard-parts:D_SOD-123-Pretty, symbol Device:D_Small
- removed J?: Connector_Generic_Conn_01x04, symbol Unified-Daughterboard-cache:Connector_Generic_Conn_01x04
- removed J? (x4): Connector_Generic_Conn_01x01, symbol Unified-Daughterboard-cache:Connector_Generic_Conn_01x01
- removed R2, R7: 22, Resistor_SMD:R_0805_2012Metric, symbol Device:R_Small
- removed R? (x2): 20k, symbol Device:R_Small
- removed R? (x4): 100k, symbol Device:R_Small
- removed R? (x4): 1k, symbol Device:R_Small
- removed U3, U4: IS31FL3733, Package_QFP:TQFP-48-1EP_7x7mm_P0.5mm_EP5x5mm, symbol random-keyboard-parts:IS31FL3733
- added Back3: MX-1U, MX_Alps_Hybrid:MX-2U, symbol MX_Alps_Hybrids:MX-1U
- added CapsLock2: MX-1U, MX_Alps_Hybrid:MX-1U-NoLED, symbol MX_Alps_Hybrids:MX-1U
- added EnterISO1: MX-1U, MX_Alps_Hybrid:MX-ISO, symbol MX_Alps_Hybrids:MX-1U
- added F13: 500mA, Fuse:Fuse_1206_3216Metric, symbol Device:Polyfuse_Small
- added LShift3: MX-1U, MX_Alps_Hybrid:MX-2.25U, symbol MX_Alps_Hybrids:MX-1U
- added Q2: 2N7002, Package_TO_SOT_SMD:SOT-23, symbol Transistor_FET:2N7002
- added R10, R11, R12, R13, R14, R15, R16, R17, R18, R19, R20, R21, R22, R23, R24, R25, R26, R27, R28, R29, R30, R31, R32, R33, R34, R35, R36, R37, R38, R39, R40, R41, R42, R43, R44, R45, R46, R47, R48, R49, R50, R51, R52, R53, R54, R55, R56, R57, R58, R59, R6, R60, R61, R62, R63, R64, R65, R66, R67, R68, R69, R70, R71, R72, R73, R74, R75, R76, R77, R78, R79, R80, R82, R83, R84, R85, R86, R87, R88, R89, R9, R90, R91: 1k, Resistor_SMD:R_0805_2012Metric, symbol Device:R_Small
- added R81, R92: 22, Resistor_SMD:R_0805_2012Metric, symbol Device:R_Small
- added U3: PRTR5V0U2X, random-keyboard-parts:SOT143B, symbol random-keyboard-parts:PRTR5V0U2X
- R4, R8: renamed from R?; footprint (none) -> Resistor_SMD:R_0805_2012Metric
- R5: value 10k -> 1k
- U2: footprint Package_QFP:TQFP-44_10x10mm_P0.8mm -> Package_DFN_QFN:QFN-44-1EP_7x7mm_P0.5mm_EP5.2x5.2mm
- USB1: renamed from USB?; footprint (none) -> Type-C:HRO-TYPE-C-31-M-12-Assembly
- renumbered Enter2 to Enter1, Enter1 to FSlash2
Connections:
- net +5V: now also A1.3 (LED), Apostrophe1.3 (LED), B1.3 (LED), BSlash1.3 (LED), Back1.3 (LED), Back2.3 (LED), C1.3 (LED), CapsLock1.3 (LED), Comma1.3 (LED), D1.3 (LED), DArrow1.3 (LED), Del1.3 (LED), E1.3 (LED), Enter1.3 (LED), Equal1.3 (LED), Esc1.3 (LED), F0.3 (LED), F1.3 (LED), F10.3 (LED), F11.3 (LED), F12.3 (LED), F2.3 (LED), F3.3 (LED), F4.3 (LED), F5.3 (LED), F6.3 (LED), F7.3 (LED), F8.3 (LED), F9.3 (LED), FSlash1.3 (LED), FSlash2.3 (LED), G1.3 (LED), H1.3 (LED), Home1.3 (LED), I1.3 (LED), J1.3 (LED), K1.3 (LED), L1.3 (LED), LAlt1.3 (LED), LArrow1.3 (LED), LBracket1.3 (LED), LCtrl1.3 (LED), LShift1.3 (LED), LShift2.3 (LED), LWK1.3 (LED), M1.3 (LED), MX0.3 (LED), MX1.3 (LED), MX2.3 (LED), MX3.3 (LED), MX4.3 (LED), MX5.3 (LED), MX6.3 (LED), MX7.3 (LED), MX8.3 (LED), MX9.3 (LED), Minus1.3 (LED), N1.3 (LED), O1.3 (LED), P1.3 (LED), Period1.3 (LED), PgDn1.3 (LED), PgUp1.3 (LED), Q1.3 (LED), R1.3 (LED), RAlt1.3 (LED), RArrow1.3 (LED), RBracket1.3 (LED), RCtrl1.3 (LED), RShift1.3 (LED), S1.3 (LED), Semicolon1.3 (LED), Space1.3 (LED), T1.3 (LED), TArrow1.3 (LED), Tab1.3 (LED), Tilda1.3 (LED), U1.3 (LED), V1.3 (LED), W1.3 (LED), X1.3 (LED), Y1.3 (LED), Z1.3 (LED), Back3.3 (LED), CapsLock2.3 (LED), EnterISO1.3 (LED), F13.1, LShift3.3 (LED)
- net COL0: now also U2.40 (PF1), CapsLock2.1 (COL), LShift3.1 (COL)
- net COL1: now also U2.37 (PF6)
- net COL10: now also F9.1 (COL), U2.25 (PD4); no longer F10.1 (COL)
- net COL11: now also F10.1 (COL), U2.22 (PD5); no longer F11.1 (COL)
- net COL12: now also Enter1.1 (COL), F11.1 (COL), LArrow1.1 (COL), RShift1.1 (COL), U2.21 (PD3); no longer F12.1 (COL)
- net COL13: now also DArrow1.1 (COL), F12.1 (COL), TArrow1.1 (COL), U2.20 (PD2), Back3.1 (COL), EnterISO1.1 (COL); no longer Enter1.1 (COL), LArrow1.1 (COL), RShift1.1 (COL)
- net COL14: now also U2.19 (PD1); no longer DArrow1.1 (COL), TArrow1.1 (COL)
- net COL15: now also U2.18 (PD0)
- net COL2: now also U2.36 (PF7)
- net COL3: now also U2.32 (PC7)
- net COL4: now also U2.31 (PC6)
- net COL5: now also U2.30 (PB6); no longer F5.1 (COL)
- net COL6: now also F5.1 (COL), U2.29 (PB5); no longer F6.1 (COL)
- net COL7: now also F6.1 (COL), U2.28 (PB4); no longer F7.1 (COL)
- net COL8: now also F7.1 (COL), U2.27 (PD7); no longer F8.1 (COL)
- net COL9: now also F8.1 (COL), U2.26 (PD6); no longer F9.1 (COL)
- net D+: now also U2.4 (D+), R92.1; no longer USB1.6 (DP1), USB1.8 (DP2)
- net D-: now also U2.3 (D-), R81.2; no longer USB1.5 (DN2), USB1.7 (DN1)
- net GND: now also Q2.2 (S), U3.1 (GND)
- net ROW0: now also U2.11 (PB3)
- net ROW1: now also U2.10 (PB2)
- net ROW2: now also U2.9 (PB1)
- net ROW3: now also U2.8 (PB0)
- net ROW4: now also U2.39 (PF4)
- net ROW5: now also U2.38 (PF5)
- net VCC: now also F13.2, U3.4 (VCC)
- net at U2.12 (PB7): now also R6.2
- net at Esc1.4 (LEDGND): now also R9.1
- net at F1.4 (LEDGND): now also R15.1
- net at Tilda1.4 (LEDGND): now also R10.1
- net at MX1.4 (LEDGND): now also R16.1
- net at F2.4 (LEDGND): now also R21.1
- net at F3.4 (LEDGND): now also R27.1
- net at MX2.4 (LEDGND): now also R22.1
- net at MX3.4 (LEDGND): now also R28.1
- net at F4.4 (LEDGND): now also R32.1
- net at F5.4 (LEDGND): now also R37.1
- net at MX4.4 (LEDGND): now also R33.1
- net at MX5.4 (LEDGND): now also R38.1
- net at F6.4 (LEDGND): now also R42.1
- net at F7.4 (LEDGND): now also R48.1
- net at MX6.4 (LEDGND): now also R43.1
- net at MX7.4 (LEDGND): now also R49.1
- net at F8.4 (LEDGND): now also R53.1
- net at F9.4 (LEDGND): now also R58.1
- net at MX8.4 (LEDGND): now also R54.1
- net at MX9.4 (LEDGND): now also R59.1
- net at F10.4 (LEDGND): now also R63.1
- net at F11.4 (LEDGND): now also R69.1
- net at MX0.4 (LEDGND): now also R64.1
- net at Minus1.4 (LEDGND): now also R70.1
- net at F12.4 (LEDGND): now also R76.1
- net at Equal1.4 (LEDGND): now also R77.1
- net at Back1.2 (ROW), D71.2 (A): now also Back3.2 (ROW)
- net at Back1.4 (LEDGND): now also Back3.4 (LEDGND), R79.1
- net at Del1.4 (LEDGND): now also R87.1
- net at Back2.4 (LEDGND): now also R84.1
- net at Home1.4 (LEDGND): now also R88.1
- net at Tab1.4 (LEDGND): now also R11.1
- net at Q1.4 (LEDGND): now also R17.1
- net at CapsLock1.2 (ROW), D4.2 (A): now also CapsLock2.2 (ROW)
- net at CapsLock1.4 (LEDGND): now also CapsLock2.4 (LEDGND), R12.1
- net at A1.4 (LEDGND): now also R18.1
- net at W1.4 (LEDGND): now also R23.1
- net at E1.4 (LEDGND): now also R29.1
- net at S1.4 (LEDGND): now also R24.1
- net at D1.4 (LEDGND): now also R30.1
- net at R1.4 (LEDGND): now also R34.1
- net at T1.4 (LEDGND): now also R39.1
- net at F0.4 (LEDGND): now also R35.1
- net at G1.4 (LEDGND): now also R40.1
- net at Y1.4 (LEDGND): now also R44.1
- net at U1.4 (LEDGND): now also R50.1
- net at H1.4 (LEDGND): now also R45.1
- net at J1.4 (LEDGND): now also R51.1
- net at I1.4 (LEDGND): now also R55.1
- net at O1.4 (LEDGND): now also R60.1
- net at K1.4 (LEDGND): now also R56.1
- net at L1.4 (LEDGND): now also R61.1
- net at P1.4 (LEDGND): now also R65.1
- net at LBracket1.4 (LEDGND): now also R71.1
- net at Semicolon1.4 (LEDGND): now also R66.1
- net at Apostrophe1.4 (LEDGND): now also R72.1
- net at RBracket1.4 (LEDGND): now also R78.1
- net at D72.2 (A), FSlash1.2 (ROW): now also EnterISO1.2 (ROW)
- net at FSlash1.4 (LEDGND): now also EnterISO1.4 (LEDGND), R80.1
- net at FSlash2.2 (ROW): now also D73.2 (A), Enter1.2 (ROW)
- net at FSlash2.4 (LEDGND): now also Enter1.4 (LEDGND), R75.1
- net at PgUp1.4 (LEDGND): now also R89.1
- net at PgDn1.4 (LEDGND): now also R90.1
- net at D5.2 (A), LShift1.2 (ROW): now also LShift3.2 (ROW)
- net at LShift1.4 (LEDGND): now also LShift3.4 (LEDGND), R13.1
- net at LCtrl1.4 (LEDGND): now also R14.1
- net at LWK1.4 (LEDGND): now also R20.1
- net at Z1.4 (LEDGND): now also R25.1
- net at X1.4 (LEDGND): now also R31.1
- net at LAlt1.4 (LEDGND): now also R26.1
- net at C1.4 (LEDGND): now also R36.1
- net at V1.4 (LEDGND): now also R41.1
- net at B1.4 (LEDGND): now also R46.1
- net at N1.4 (LEDGND): now also R52.1
- net at Space1.4 (LEDGND): now also R47.1
- net at M1.4 (LEDGND): now also R57.1
- net at Comma1.4 (LEDGND): now also R62.1
- net at Period1.4 (LEDGND): now also R67.1
- net at BSlash1.4 (LEDGND): now also R73.1
- net at RAlt1.4 (LEDGND): now also R68.1
- net at RCtrl1.4 (LEDGND): now also R74.1
- net at RShift1.4 (LEDGND): now also R82.1
- net at LArrow1.4 (LEDGND): now also R83.1
- net at TArrow1.4 (LEDGND): now also R85.1
- net at DArrow1.4 (LEDGND): now also R86.1
- net at RArrow1.4 (LEDGND): now also R91.1
- net at LShift2.4 (LEDGND): now also R19.1
- new net: Q2.1 (G), R6.1
- new net: R81.1, U3.3 (IO2), USB1.5 (DN2), USB1.7 (DN1)
- new net: R92.2, U3.2 (IO1), USB1.6 (DP1), USB1.8 (DP2)
- new net LEDGND: Q2.3 (D), R10.2, R11.2, R12.2, R13.2, R14.2, R15.2, R16.2, R17.2, R18.2, R19.2, R20.2, R21.2, R22.2, R23.2, R24.2, R25.2, R26.2, R27.2, R28.2, R29.2, R30.2, R31.2, R32.2, R33.2, R34.2, R35.2, R36.2, R37.2, R38.2, R39.2, R40.2, R41.2, R42.2, R43.2, R44.2, R45.2, R46.2, R47.2, R48.2, R49.2, R50.2, R51.2, R52.2, R53.2, R54.2, R55.2, R56.2, R57.2, R58.2, R59.2, R60.2, R61.2, R62.2, R63.2, R64.2, R65.2, R66.2, R67.2, R68.2, R69.2, R70.2, R71.2, R72.2, R73.2, R74.2, R75.2, R76.2, R77.2, R78.2, R79.2, R80.2, R82.2, R83.2, R84.2, R85.2, R86.2, R87.2, R88.2, R89.2, R9.2, R90.2, R91.2
- no-connect marks 0 -> 2
Other:
- moved on the sheet: A1, Apostrophe1, B1, BSlash1, Back1, Back2, C1, C2, C3, C4, C5, C6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
